File: FuzzTester/Kicad/Fuzz.kicad_pcb (KiCad board)
At the start: 2 copper layers, 180 x 100 mm, 133 parts, among them J1 Audio In/Out JST XH, J10 Key Pad JST XH, J11 1602 LCD JST XH, J2 POT B10K JST XH, J3 POT B5K JST XH, J4 VOL POT A100K JST XH, J5 TestPower_PinHeader, J6 9V Power JST XH, J7 Boot Reset PinHeader, J8 SPI Test PinHeader, J9 SWD_PinHeader, Q1 PN2222A, Q10 2SC1815, Q11 S8050, Q12 S9013, Q13 S9014, Q14 S9018, Q15 BC848B, Q16 2SC1623, Q17 MPSA18, Q18 MPSA18, Q19 2N5088, Q2 MMBT3904, Q20 2N5088, Q21 PN2222A, Q22 MMBT3904, Q23 MMBT5551L, Q24 MMBTA42, Q25 BC807, Q26 BC846, Q27 BC847B, Q28 BC847C, Q29 C945, Q3 MMBT5551L, Q30 2SC1815, Q31 S8050, Q32 S9013, Q33 S9014, Q34 S9018, Q35 BC848B, Q36 2SC1623, Q37 MPSA18, Q38 MPSA18, Q39 2N5088, Q4 MMBTA42, Q40 2N5088, Q5 BC807, Q6 BC846, Q7 BC847B, Q8 BC847C, Q9 C945, U1 AMS1117-5.0, U10 CD4052B, U11 CD4052B, U12 CD4052B, U13 CD4052B, U14 CD4051B, U15 CD4052B, U16 CD4051B, U17 CD4052B, U18 CD4052B, U19 CD4052B, U2 AMS1117-3.3, U20 74HC595, U21 CD4051B, U3 STM32F103C8Tx, U4 CD4051B, U5 74HC595, U6 CD4052B, U7 CD4051B, U8 CD4052B, U9 CD4051B, Y1 8MHz

Commit message: PCB fixes
Routing:
- net GND: track 1435.1 -> 1375.7 mm, vias 54 -> 55
- net +5V: track 606.9 -> 571.7 mm, vias 21 -> 24
- net Net-(C1-Pad1): track 57.0 -> 54.2 mm
- net /TRANSISTOR_B_GROUP_SELECTION_0: track 60.3 -> 61.0 mm
