File: FuzzTester/Kicad/Fuzz.kicad_pcb (KiCad board)
At the start: 2 copper layers, 100 x 82 mm, 142 parts, among them J1 Audio In/Out JST XH, J10 Key Pad JST XH, J11 LCD JST XH, J12 Bypass Switch JST XH, J2 POT B10K JST XH, J3 POT B5K JST XH, J4 VOL POT A100K JST XH, J5 PowerTest_PinHeader, J6 9V Power JST XH, J7 Boot Reset PinHeader, J8 SPI Test PinHeader, J9 SWD_PinHeader, Q1 PN2222A, Q10 2SC1815, Q11 S8050, Q12 S9013, Q13 S9014, Q14 S9018, Q15 BC848B, Q16 2SC1623, Q17 MPSA18, Q18 MPSA18, Q19 2N5088, Q2 MMBT3904, Q20 2N5088, Q21 PN2222A, Q22 MMBT3904, Q23 MMBT5551L, Q24 MMBTA42, Q25 BC807, Q26 BC846, Q27 BC847B, Q28 BC847C, Q29 C945, Q3 MMBT5551L, Q30 2SC1815, Q31 S8050, Q32 S9013, Q33 S9014, Q34 S9018, Q35 BC848B, Q36 2SC1623, Q37 MPSA18, Q38 MPSA18, Q39 2N5088, Q4 MMBTA42, Q40 2N5088, Q5 BC807, Q6 BC846, Q7 BC847B, Q8 BC847C, Q9 C945, U1 AMS1117-5.0, U10 CD4052B, U11 CD4052B, U12 CD4052B, U13 CD4052B, U14 CD4051B, U15 CD4052B, U16 CD4051B, U17 CD4052B, U18 CD4052B, U19 CD4052B, U2 AMS1117-3.3, U20 74HC595, U21 CD4051B, U22 4504, U23 4504, U24 4504, U25 CD4053B, U3 STM32F103C8Tx, U4 CD4051B, U5 74HC595, U6 CD4052B, U7 CD4051B, U8 CD4052B, U9 CD4051B, Y1 8MHz

Commit message: 9V
Parts:
- moved C35 14.9 mm to (39.6, 103.6), turned to 90 degrees
- moved C25 13.4 mm to (54.6, 58.5), turned to 90 degrees
- moved C45 13.4 mm to (54.6, 47.5), turned to 90 degrees
- moved C11 13.4 mm to (88.9, 47.5), turned to 90 degrees
- moved C20 13.4 mm to (54.6, 69.4), turned to 90 degrees
- moved C22 13.4 mm to (66.0, 47.5), turned to 90 degrees
- moved C24 13.4 mm to (77.5, 58.4), turned to 90 degrees
- moved C26 13.4 mm to (66.0, 69.4), turned to 90 degrees
- moved C27 13.4 mm to (77.5, 69.4), turned to 90 degrees
- moved C28 13.4 mm to (77.5, 47.5), turned to 90 degrees
- moved C29 13.4 mm to (66.0, 85.9), turned to 90 degrees
- moved C30 13.4 mm to (77.5, 96.8), turned to 90 degrees
- moved C33 13.4 mm to (66.0, 107.7), turned to 90 degrees
- moved C34 13.4 mm to (77.5, 107.7), turned to 90 degrees
- moved C21 13.4 mm to (77.5, 85.8), turned to 90 degrees
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Routing:
- net +9V: track 74.1 -> 371.4 mm, vias 3 -> 25
- net GND: track 27.3 -> 115.9 mm, vias 6 -> 30
- net /Mcu/BYPASS_SWITCH_3V3: track 60.6 -> 0.00 mm, vias 3 -> 0
- net /ShiftRegistersCD/COMPONENT_SELECTION_INPUT: track 0.00 -> 50.2 mm, vias 0 -> 2
- net +5V: track 79.4 -> 123.0 mm, vias 1 -> 3
- net /AudioInOut/JACK_IN_SIGNAL: track 32.0 -> 0.00 mm, vias 3 -> 0
- net /TRANSISTOR_C_GROUP_SELECTION_3V3_0: track 0.00 -> 23.9 mm, vias 0 -> 2
- net /1602_BACK_LIGHT_PIN_2: track 21.8 -> 0.00 mm
- net /1602_BACK_LIGHT_PIN_1: track 20.0 -> 0.00 mm, vias 2 -> 0
- net /TRANSISTOR_C_GROUP_SELECTION_3V3_2: track 0.00 -> 19.4 mm
- net /TRANSISTOR_C_GROUP_SELECTION_3V3_1: track 0.00 -> 18.7 mm
- net /CAPACITOR_D_SELECTION_3V3_2: track 0.00 -> 16.9 mm, vias 0 -> 2
- net /TRANSISTOR_C_SELECTION_3V3_0: track 0.00 -> 15.7 mm, vias 0 -> 2
- net +3V3: track 72.4 -> 88.0 mm, vias 4 -> 8
- net /TRANSISTOR_C_SELECTION_3V3_1: track 0.00 -> 14.6 mm, vias 0 -> 2
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
Commit message: More traces
Routing:
- net +3V3: track 88.0 -> 197.6 mm, vias 8 -> 12
- net /TransistorsC/BASE: track 0.00 -> 97.1 mm, vias 0 -> 4
- net /CAPACITOR_A_SELECTION_1: track 0.00 -> 76.4 mm, vias 0 -> 2
- net /CAPACITOR_A_SELECTION_0: track 0.00 -> 72.3 mm, vias 0 -> 2
- net /TRANSISTOR_B_GROUP_SELECTION_2: track 0.00 -> 69.7 mm, vias 0 -> 4
- net /CAPACITOR_A_SELECTION_2: track 0.00 -> 69.4 mm, vias 0 -> 2
- net /TRANSISTOR_B_GROUP_SELECTION_1: track 0.00 -> 67.5 mm, vias 0 -> 6
- net /TRANSISTOR_B_SELECTION_1: track 0.00 -> 62.6 mm, vias 0 -> 4
- net /Mcu/BYPASS_SWITCH_3V3: track 0.00 -> 60.4 mm, vias 0 -> 3
- net /TRANSISTOR_B_GROUP_SELECTION_0: track 0.00 -> 60.1 mm, vias 0 -> 5
- net /BYPASS_MODE: track 0.00 -> 59.7 mm, vias 0 -> 4
- net /TransistorsB/TG_1_COLLECTOR: track 0.00 -> 55.8 mm, vias 0 -> 2
- net /AudioInOut/JACK_OUT_SIGNAL: track 0.00 -> 51.3 mm, vias 0 -> 1
- net /JACK_OUT_SIGNAL_FROM_FUZZ: track 0.00 -> 47.8 mm, vias 0 -> 1
- net /AudioInOut/JACK_IN_SIGNAL: track 0.00 -> 45.1 mm, vias 0 -> 1
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
Commit message: Transistors C almost done
Parts:
- moved U5 0.06 mm to (60.5, 66.0)
Routing:
- net GND: track 116.9 -> 938.6 mm, vias 31 -> 41
- net /TransistorsC/EMITTER: track 0.00 -> 218.9 mm, vias 0 -> 9
- net /CapacitorsD/CAPACITOR_AUDIO_OUTPUT: track 0.00 -> 127.4 mm
- net /CapacitorsD/CAPACITOR_AUDIO_INPUT: track 0.00 -> 108.4 mm, vias 0 -> 5
- net /TransistorsC/TG_1_COLLECTOR: track 0.00 -> 105.0 mm, vias 0 -> 10
- net /TRANSISTOR_C_SELECTION_0: track 9.83 -> 112.6 mm, vias 0 -> 8
- net /TRANSISTOR_C_SELECTION_1: track 8.58 -> 110.1 mm, vias 0 -> 8
- net /TransistorsC/18_COLLECTOR: track 0.00 -> 85.1 mm, vias 0 -> 1
- net /TransistorsC/18_BASE: track 0.00 -> 85.1 mm, vias 0 -> 2
- net /TransistorsC/17_BASE: track 0.00 -> 78.1 mm, vias 0 -> 1
- net /TransistorsC/17_COLLECTOR: track 0.00 -> 76.5 mm, vias 0 -> 2
- net /TransistorsC/15_BASE: track 0.00 -> 70.7 mm, vias 0 -> 2
- net /TransistorsC/19_BASE: track 0.00 -> 69.5 mm, vias 0 -> 3
- net /TransistorsC/15_COLLECTOR: track 0.00 -> 67.1 mm, vias 0 -> 2
- net /TransistorsC/19_COLLECTOR: track 0.00 -> 66.4 mm, vias 0 -> 2
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