File: FuzzTester/Kicad/ShiftRegisters.sch (KiCad schematic (older format))
At the start: 2 parts, among them U5 74HC595

Commit message: PCB Placement 100x82
Connections:
- net +5V: no longer C20.1, U5.16 (VCC)
- new net +3V3: C20.1, U5.16 (VCC)
Other:
- note added: "Shift Register"
- note removed: "Shift Register: Transistor/Capacitor Selection\n\n"
- moved on the sheet: C35, U20
Changed lines of the file:
@@
 $Descr A4 11693 8268
 encoding utf-8
-Sheet 7 9
+Sheet 5 11
 Title "Guitar Pedal Effect Fuzz Digitally Controlled"
 Date "2020-04-07"
@@
 Comment4 "Shift Register for either A capacitors/B transistors or C transistors/D capacitors"
 $EndDescr
-Text Notes 3900 1700 0    50   ~ 10
-Shift Register: Transistor/Capacitor Selection\n\n
-Wire Wire Line
-	3650 2850 4150 2850
-Wire Wire Line
-	4550 1900 4550 2350
-Wire Wire Line
-	4850 1900 4550 1900
+Text HLabel 5050 2600 0    50   Input ~ 0
+COMPONENT_SELECTION_INPUT
+Text HLabel 5850 3500 2    50   Input ~ 0
+COMPONENT_SELECTION_OUTPUT
+$Comp
+L power:+5V #PWR032
+U 1 1 5EB6323A
+P 4550 2900
+AR Path="/5E87C69B/5EB6323A" Ref="#PWR032"  Part="1"
+AR Path="/5EB914C2/5EB6323A" Ref="#PWR?"  Part="1"
+AR Path="/5EB9C150/5EB6323A" Ref="#PWR?"  Part="1"
+AR Path="/5F697325/5EB6323A" Ref="#PWR?"  Part="1"
+AR Path="/5F99B130/5EB6323A" Ref="#PWR093"  Part="1"
+F 0 "#PWR093" H 4550 2750 50  0001 C CNN
+F 1 "+5V" H 4565 3073 50  0000 C CNN
+F 2 "" H 4550 2900 50  0001 C CNN
+F 3 "" H 4550 2900 50  0001 C CNN
+	1    4550 2900
+	1    0    0    -1
+$EndComp
+Text HLabel 5850 3300 2    50   Input ~ 0
+CAPACITOR_SELECTION_2
+Text HLabel 5850 3200 2    50   Input ~ 0
+CAPACITOR_SELECTION_1
+Text HLabel 5850 3100 2    50   Input ~ 0
+CAPACITOR_SELECTION_0
+Text HLabel 5850 3000 2    50   Input ~ 0
+TRANSISTOR_SELECTION_1
+Text HLabel 5850 2900 2    50   Input ~ 0
+TRANSISTOR_SELECTION_0
+Text HLabel 5850 2800 2    50   Input ~ 0
+TRANSISTOR_GROUPS_SELECTION_2
+Text HLabel 5850 2700 2    50   Input ~ 0
+TRANSISTOR_GROUPS_SELECTION_1
+Text HLabel 5850 2600 2    50   Input ~ 0
+TRANSISTOR_GROUPS_SELECTION_0
+Text HLabel 5050 3100 0    50   Input ~ 0
+GPIO_LATCH
+Text HLabel 5050 2800 0    50   Input ~ 0
+SPI2_CSK
+$Comp
+L 74xx:74HC595 U5
+U 1 1 5EB63229
+P 5450 3000
+AR Path="/5E87C69B/5EB63229" Ref="U5"  Part="1"
+AR Path="/5EB914C2/5EB63229" Ref="U?"  Part="1"
+AR Path="/5EB9C150/5EB63229" Ref="U?"  Part="1"
+AR Path="/5F697325/5EB63229" Ref="U?"  Part="1"
+AR Path="/5F99B130/5EB63229" Ref="U20"  Part="1"
+F 0 "U20" H 5450 3781 50  0000 C CNN
+F 1 "74HC595" H 5450 3690 50  0000 C CNN
+F 2 "Package_SO:SOIC-16_3.9x9.9mm_P1.27mm" H 5450 3000 50  0001 C CNN
+F 3 "http://www.ti.com/lit/ds/symlink/sn74hc595.pdf" H 5450 3000 50  0001 C CNN
+	1    5450 3000
+	1    0    0    -1
+$EndComp
+$Comp
+L power:GND #PWR033
+U 1 1 5EB63223
+P 5050 3200
+AR Path="/5E87C69B/5EB63223" Ref="#PWR033"  Part="1"
+AR Path="/5EB914C2/5EB63223" Ref="#PWR?"  Part="1"
+AR Path="/5EB9C150/5EB63223" Ref="#PWR?"  Part="1"
+AR Path="/5F697325/5EB63223" Ref="#PWR?"  Part="1"
+AR Path="/5F99B130/5EB63223" Ref="#PWR094"  Part="1"
+F 0 "#PWR094" H 5050 2950 50  0001 C CNN
+F 1 "GND" H 5055 3027 50  0000 C CNN
+F 2 "" H 5050 3200 50  0001 C CNN
+F 3 "" H 5050 3200 50  0001 C CNN
+	1    5050 3200
+	1    0    0    -1
+$EndComp
+$Comp
+L power:GND #PWR035
+U 1 1 5EB6321D
+P 5450 3700
+AR Path="/5E87C69B/5EB6321D" Ref="#PWR035"  Part="1"
+AR Path="/5EB914C2/5EB6321D" Ref="#PWR?"  Part="1"
+AR Path="/5EB9C150/5EB6321D" Ref="#PWR?"  Part="1"
+AR Path="/5F697325/5EB6321D" Ref="#PWR?"  Part="1"
+AR Path="/5F99B130/5EB6321D" Ref="#PWR096"  Part="1"
+F 0 "#PWR096" H 5450 3450 50  0001 C CNN
+F 1 "GND" H 5455 3527 50  0000 C CNN
+F 2 "" H 5450 3700 50  0001 C CNN
+F 3 "" H 5450 3700 50  0001 C CNN
+	1    5450 3700
+	1    0    0    -1
+$EndComp
+$Comp
+L power:GND #PWR036
+U 1 1 5EB63210
+P 5750 2250
+AR Path="/5E87C69B/5EB63210" Ref="#PWR036"  Part="1"
+AR Path="/5EB914C2/5EB63210" Ref="#PWR?"  Part="1"
+AR Path="/5EB9C150/5EB63210" Ref="#PWR?"  Part="1"
+AR Path="/5F697325/5EB63210" Ref="#PWR?"  Part="1"
+AR Path="/5F99B130/5EB63210" Ref="#PWR097"  Part="1"
+F 0 "#PWR097" H 5750 2000 50  0001 C CNN
+F 1 "GND" H 5755 2077 50  0000 C CNN
+F 2 "" H 5750 2250 50  0001 C CNN
+F 3 "" H 5750 2250 50  0001 C CNN
+	1    5750 2250
+	1    0    0    -1
+$EndComp
 $Comp
 L Device:C C20
 U 1 1 5EB6320A
-P 4850 2050
+P 5750 2100
 AR Path="/5E87C69B/5EB6320A" Ref="C20"  Part="1"
 AR Path="/5EB914C2/5EB6320A" Ref="C?"  Part="1"
@@
 AR Path="/5F697325/5EB6320A" Ref="C?"  Part="1"
 AR Path="/5F99B130/5EB6320A" Ref="C35"  Part="1"
-F 0 "C35" H 4965 2096 50  0000 L CNN
-F 1 "100nF" H 4965 2005 50  0000 L CNN
-F 2 "Capacitor_SMD:C_0805_2012Metric_Pad1.15x1.40mm_HandSolder" H 4888 1900 50  0001 C CNN
-F 3 "~" H 4850 2050 50  0001 C CNN
-	1    4850 2050
+F 0 "C35" H 5865 2146 50  0000 L CNN
+F 1 "100nF" H 5865 2055 50  0000 L CNN
+F 2 "Capacitor_SMD:C_0805_2012Metric_Pad1.15x1.40mm_HandSolder" H 5788 1950 50  0001 C CNN
+F 3 "~" H 5750 2100 50  0001 C CNN
+	1    5750 2100
 	1    0    0    -1
 $EndComp
+Wire Wire Line
+	5750 1950 5450 1950
+Wire Wire Line
+	5450 1950 5450 2400
+Wire Wire Line
+	4550 2900 5050 2900
 $Comp
-L power:GND #PWR036
-U 1 1 5EB63210
-P 4850 2200
-AR Path="/5E87C69B/5EB63210" Ref="#PWR036"  Part="1"
-AR Path="/5EB914C2/5EB63210" Ref="#PWR?"  Part="1"
-AR Path="/5EB9C150/5EB63210" Ref="#PWR?"  Part="1"
-AR Path="/5F697325/5EB63210" Ref="#PWR?"  Part="1"
-AR Path="/5F99B130/5EB63210" Ref="#PWR097"  Part="1"
-F 0 "#PWR097" H 4850 1950 50  0001 C CNN
-F 1 "GND" H 4855 2027 50  0000 C CNN
-F 2 "" H 4850 2200 50  0001 C CNN
-F 3 "" H 4850 2200 50  0001 C CNN
-	1    4850 2200
+L power:+3V3 #PWR0116
+U 1 1 5EDC7BE8
+P 5450 1950
+AR Path="/5E87C69B/5EDC7BE8" Ref="#PWR0116"  Part="1"
+AR Path="/5F99B130/5EDC7BE8" Ref="#PWR0118"  Part="1"
+F 0 "#PWR0118" H 5450 1800 50  0001 C CNN
+F 1 "+3V3" H 5465 2123 50  0000 C CNN
+F 2 "" H 5450 1950 50  0001 C CNN
+F 3 "" H 5450 1950 50  0001 C CNN
+	1    5450 1950
 	1    0    0    -1
 $EndComp
-Connection ~ 4550 1900
-$Comp
-L power:+5V #PWR034
-U 1 1 5EB63217
-P 4550 1900
-AR Path="/5E87C69B/5EB63217" Ref="#PWR034"  Part="1"
-AR Path="/5EB914C2/5EB63217" Ref="#PWR?"  Part="1"
-AR Path="/5EB9C150/5EB63217" Ref="#PWR?"  Part="1"
-AR Path="/5F697325/5EB63217" Ref="#PWR?"  Part="1"
-AR Path="/5F99B130/5EB63217" Ref="#PWR095"  Part="1"
-F 0 "#PWR095" H 4550 1750 50  0001 C CNN
-F 1 "+5V" H 4565 2073 50  0000 C CNN
-F 2 "" H 4550 1900 50  0001 C CNN
-F 3 "" H 4550 1900 50  0001 C CNN
-	1    4550 1900
-	1    0    0    -1
-$EndComp
-$Comp
-L power:GND #PWR035
-U 1 1 5EB6321D
-P 4550 3650
-AR Path="/5E87C69B/5EB6321D" Ref="#PWR035"  Part="1"
-AR Path="/5EB914C2/5EB6321D" Ref="#PWR?"  Part="1"
-AR Path="/5EB9C150/5EB6321D" Ref="#PWR?"  Part="1"
-AR Path="/5F697325/5EB6321D" Ref="#PWR?"  Part="1"
-AR Path="/5F99B130/5EB6321D" Ref="#PWR096"  Part="1"
-F 0 "#PWR096" H 4550 3400 50  0001 C CNN
-F 1 "GND" H 4555 3477 50  0000 C CNN
-F 2 "" H 4550 3650 50  0001 C CNN
-F 3 "" H 4550 3650 50  0001 C CNN
-	1    4550 3650
-	1    0    0    -1
-$EndComp
-$Comp
-L power:GND #PWR033
-U 1 1 5EB63223
-P 4150 3150
-AR Path="/5E87C69B/5EB63223" Ref="#PWR033"  Part="1"
-AR Path="/5EB914C2/5EB63223" Ref="#PWR?"  Part="1"
-AR Path="/5EB9C150/5EB63223" Ref="#PWR?"  Part="1"
-AR Path="/5F697325/5EB63223" Ref="#PWR?"  Part="1"
-AR Path="/5F99B130/5EB63223" Ref="#PWR094"  Part="1"
-F 0 "#PWR094" H 4150 2900 50  0001 C CNN
-F 1 "GND" H 4155 2977 50  0000 C CNN
-F 2 "" H 4150 3150 50  0001 C CNN
-F 3 "" H 4150 3150 50  0001 C CNN
-	1    4150 3150
-	1    0    0    -1
-$EndComp
-$Comp
-L 74xx:74HC595 U5
-U 1 1 5EB63229
-P 4550 2950
-AR Path="/5E87C69B/5EB63229" Ref="U5"  Part="1"
-AR Path="/5EB914C2/5EB63229" Ref="U?"  Part="1"
-AR Path="/5EB9C150/5EB63229" Ref="U?"  Part="1"
-AR Path="/5F697325/5EB63229" Ref="U?"  Part="1"
-AR Path="/5F99B130/5EB63229" Ref="U20"  Part="1"
-F 0 "U20" H 4550 3731 50  0000 C CNN
-F 1 "74HC595" H 4550 3640 50  0000 C CNN
-F 2 "Package_SO:SOIC-16_3.9x9.9mm_P1.27mm" H 4550 2950 50  0001 C CNN
-F 3 "http://www.ti.com/lit/ds/symlink/sn74hc595.pdf" H 4550 2950 50  0001 C CNN
-	1    4550 2950
-	1    0    0    -1
-$EndComp
-Text HLabel 4150 2750 0    50   Input ~ 0
-SPI2_CSK
-Text HLabel 4150 3050 0    50   Input ~ 0
-GPIO_LATCH
-Text HLabel 4950 2550 2    50   Input ~ 0
-TRANSISTOR_GROUPS_SELECTION_0
-Text HLabel 4950 2650 2    50   Input ~ 0
-TRANSISTOR_GROUPS_SELECTION_1
-Text HLabel 4950 2750 2    50   Input ~ 0
-TRANSISTOR_GROUPS_SELECTION_2
-Text HLabel 4950 2850 2    50   Input ~ 0
-TRANSISTOR_SELECTION_0
-Text HLabel 4950 2950 2    50   Input ~ 0
-TRANSISTOR_SELECTION_1
-Text HLabel 4950 3050 2    50   Input ~ 0
-CAPACITOR_SELECTION_0
-Text HLabel 4950 3150 2    50   Input ~ 0
-CAPACITOR_SELECTION_1
-Text HLabel 4950 3250 2    50   Input ~ 0
-CAPACITOR_SELECTION_2
-$Comp
-L power:+5V #PWR032
-U 1 1 5EB6323A
-P 3650 2850
-AR Path="/5E87C69B/5EB6323A" Ref="#PWR032"  Part="1"
-AR Path="/5EB914C2/5EB6323A" Ref="#PWR?"  Part="1"
-AR Path="/5EB9C150/5EB6323A" Ref="#PWR?"  Part="1"
-AR Path="/5F697325/5EB6323A" Ref="#PWR?"  Part="1"
-AR Path="/5F99B130/5EB6323A" Ref="#PWR093"  Part="1"
-F 0 "#PWR093" H 3650 2700 50  0001 C CNN
-F 1 "+5V" H 3665 3023 50  0000 C CNN
-F 2 "" H 3650 2850 50  0001 C CNN
-F 3 "" H 3650 2850 50  0001 C CNN
-	1    3650 2850
-	1    0    0    -1
-$EndComp
-Text HLabel 4950 3450 2    50   Input ~ 0
-COMPONENT_SELECTION_OUTPUT
-Text HLabel 4150 2550 0    50   Input ~ 0
-COMPONENT_SELECTION_INPUT
+Connection ~ 5450 1950
+Text Notes 5200 1550 0    50   ~ 10
+Shift Register
+Wire Notes Line
+	7500 1350 7500 4200
+Wire Notes Line
+	7500 4200 3500 4200
+Wire Notes Line
+	3500 4200 3500 1350
+Wire Notes Line
+	3500 1350 7500 1350
 $EndSCHEMATC
