File: Kicad/3_Stm32DevBoard/Mcu.sch (KiCad schematic (older format))
At the start: 21 parts, among them J10 JST XH Buttons, J11 LCD JST XH, J12 Bypass Switch JST XH, J3 Jumper BOOT0, J7 UART Pin Header, J8 Jumper BOOT1, J9 SWD, SW1 RESET, U3 STM32F103C8Tx, Y1 8MHz

Commit message: STM32 Dev Board
Parts:
- removed C10, C7, C8, C9: 100nF, Capacitor_SMD:C_0805_2012Metric_Pad1.15x1.40mm_HandSolder, symbol Device:C
- removed C20: 10uF, Capacitor_SMD:C_0805_2012Metric_Pad1.15x1.40mm_HandSolder, symbol Device:C
- removed C5, C6: 20pF, Capacitor_SMD:C_0805_2012Metric_Pad1.15x1.40mm_HandSolder, symbol Device:C
- removed J3: Jumper BOOT0, Connector_PinHeader_2.54mm:PinHeader_1x03_P2.54mm_Vertical, symbol Connector:Conn_01x03_Male
- removed J8: Jumper BOOT1, Connector_PinHeader_2.54mm:PinHeader_1x03_P2.54mm_Vertical, symbol Connector:Conn_01x03_Male
- removed J9: SWD, Connector_PinHeader_2.54mm:PinHeader_1x06_P2.54mm_Vertical, symbol Connector:Conn_01x06_Male
- removed R7: 10K, Resistor_SMD:R_0805_2012Metric_Pad1.15x1.40mm_HandSolder, symbol Device:R
- removed RN2: 33R, Resistor_SMD:R_Array_Convex_4x0603, symbol Device:R_Pack04
- removed SW1: RESET, Button_Switch_SMD:SW_SPST_CK_RS282G05A3, symbol Switch:SW_SPST
- removed U3: STM32F103C8Tx, Package_QFP:LQFP-48-1EP_7x7mm_P0.5mm_EP3.6x3.6mm_ThermalVias, symbol MCU_ST_STM32F1:STM32F103C8Tx
- removed Y1: 8MHz, Crystal:Crystal_HC49-4H_Vertical, symbol Device:Crystal
- added U3: ChinaBluePill, 3_Stm32DevBoard:BluePill_STM32F103C, symbol STM32a:ChinaBluePill
- R5: value 220R -> 33R
- R6: value 10K -> 33R
Connections:
- net labels removed: 3V3, BOOT0, BOOT1, MCU_BYPASS_CAPS, NRST, OSC_IN, OSC_OUT, SYS_JTDO_TRACESWO, SYS_JTICK_SWCLK, SYS_JTICK_SWCLK_MCU, SYS_JTMS_SWDIO, SYS_JTMS_SWDIO_MCU
- wire segments 109 -> 40
- no-connect marks 9 -> 13
Other:
- note removed: "Boot 0\n"
- note removed: "Boot 1\n"
- note removed: "Check: Concave or Convex footprint"
- note removed: "Cl = 2 * (CLOAD_CRYSTAL - CPARASITIC)\n (for STM32F405...)\n = 2 * (9pF - 2pF) = 14 pF \n(see YouTube: KiCad STM32 Hardware Design \nand JLCPCB Assembly)\n"
- note removed: "Micro Controller Unit Bypass Capacitors\n\n\n\n"
- note removed: "Oscillator\n\n\n"
- note removed: "Resistor for driving less and\nremoving high frequenties\n(see same YouTube video\nas above)"
- note removed: "SWD\n\n\n"
- note removed: "f(-3dB) = 1/(2*pi*C*R)\n= 16 MHz * 2 * pi * 9 pF * R) = 1 <=> R ="
- note removed: "https://vivonomicon.com/2018/05/05/your-own-hardware-designing-an-stm32-development-board/"
- moved on the sheet: J10, J11, J12, J7
